Commit message: Appearance Update

File: Hector_ROS_Simulation/hector_description/xacro/gazebo.xacro (robot description, xacro)
@@ -73,5 +73,5 @@
         <kp  value="100000.0"/>
         <kd  value="1000.0"/>
-        <material>Gazebo/DarkGrey</material>
+        <material>Gazebo/Grey</material>
     </gazebo>
     <gazebo reference="L_hip2">
@@ -80,5 +80,5 @@
         <kp  value="100000.0"/>
         <kd  value="1000.0"/>
-        <material>Gazebo/Red</material>
+        <material>Gazebo/Grey</material>
     </gazebo>
     <gazebo reference="L_thigh">
@@ -88,5 +88,5 @@
         <kd  value="1000.0"/>
         <self_collide>0</self_collide>
-        <material>Gazebo/DarkGrey</material>
+        <material>Gazebo/Grey</material>
     </gazebo>
     <gazebo reference="L_calf">
@@ -96,4 +96,5 @@
         <kd  value="1000.0"/>
         <self_collide>0</self_collide>
+        <material>Gazebo/Grey</material>
     </gazebo>
     <gazebo reference="L_toe">
@@ -103,5 +104,5 @@
         <kd  value="1000.0"/>
         <self_collide>0</self_collide>
-        <material>Gazebo/DarkGrey</material>
+        <material>Gazebo/Grey</material>
     </gazebo>
     <!--R leg -->
@@ -111,5 +112,5 @@
         <kp  value="100000.0"/>
         <kd  value="1000.0"/>
-        <material>Gazebo/DarkGrey</material>
+        <material>Gazebo/Grey</material>
     </gazebo>
     <gazebo reference="R_hip2">
@@ -118,5 +119,5 @@
         <kp  value="100000.0"/>
         <kd  value="1000.0"/>
-        <material>Gazebo/Red</material>
+        <material>Gazebo/Grey</material>
     </gazebo>
     <gazebo reference="R_thigh">
@@ -126,5 +127,5 @@
         <kd  value="1000.0"/>
         <self_collide>0</self_collide>
-        <material>Gazebo/DarkGrey</material>
+        <material>Gazebo/Grey</material>
     </gazebo>
     <gazebo reference="R_calf">
@@ -134,4 +135,5 @@
         <kd  value="1000.0"/>
         <self_collide>0</self_collide>
+        <material>Gazebo/Grey</material>
     </gazebo>
     <gazebo reference="R_toe">
@@ -141,5 +143,5 @@
         <kd  value="1000.0"/>
         <self_collide>0</self_collide>
-        <material>Gazebo/DarkGrey</material>
+        <material>Gazebo/Grey</material>
     </gazebo>
 </robot>
