Commit message: arm controller

File: Hector_ROS_Simulation/hector_description/xacro/arm.xacro (robot description, xacro)
@@ -1,4 +1,5 @@
 <?xml version="1.0"?>
 <robot xmlns:xacro="http://www.ros.org/wiki/xacro">
+<xacro:include filename="$(find hector_description)/xacro/arm_transmission.xacro"/>
     <xacro:macro name="arm" params="name mirror mirror_dae  *origin">
         <joint name="${name}_twist_joint" type="revolute">
@@ -14,8 +15,8 @@
             <dynamics damping="${damping}" friction="${friction}"/>
             <xacro:if value="${(mirror_dae == True)}">
-                <limit effort="${twist_torque_max}" velocity="${twist_velocity_max}" lower="${twist_min*PI/180.0}" upper="${twist_max*PI/180.0}"/>
+                <limit effort="${twist_torque_max}" velocity="${twist_velocity_max}" lower="${twist_min}" upper="${twist_max}"/>
             </xacro:if>
             <xacro:if value="${(mirror_dae == False)}">
-                <limit effort="${twist_torque_max}" velocity="${twist_velocity_max}" lower="${-twist_max*PI/180.0}" upper="${-twist_min*PI/180.0}"/>
+                <limit effort="${twist_torque_max}" velocity="${twist_velocity_max}" lower="${-twist_max}" upper="${-twist_min}"/>
             </xacro:if>
         </joint>
@@ -59,5 +60,5 @@
             <axis xyz="0 1 0"/>
             <dynamics damping="${damping}" friction="${friction}"/>
-            <limit effort="${shoulder_torque_max}" velocity="${shoulder_velocity_max}" lower="${shoulder_min*PI/180.0}" upper="${shoulder_max*PI/180.0}"/>
+            <limit effort="${shoulder_torque_max}" velocity="${shoulder_velocity_max}" lower="${shoulder_min}" upper="${shoulder_max}"/>
         </joint>
         <link name="${name}_shoulder">
@@ -97,5 +98,5 @@
             <axis xyz="0 1 0"/>
             <dynamics damping="${damping}" friction="${friction}"/>
-            <limit effort="${elbow_torque_max}" velocity="${elbow_velocity_max}" lower="${elbow_min*PI/180.0}" upper="${elbow_max*PI/180.0}"/>
+            <limit effort="${elbow_torque_max}" velocity="${elbow_velocity_max}" lower="${elbow_min}" upper="${elbow_max}"/>
         </joint>
         <link name="${name}_elbow">
@@ -122,4 +123,5 @@
             </inertial>
         </link>
+        <xacro:arm_transmission name="${name}"/>
     </xacro:macro>
 </robot>

File: Hector_ROS_Simulation/hector_description/xacro/transmission.xacro (robot description, xacro)
@@ -53,3 +53,36 @@
         </transmission>
     </xacro:macro>
+    <xacro:macro name="arm_transmission" params="name">
+        <!--Left arm  -->
+        <transmission name="${name}_twist_tran">
+            <type>transmission_interface/SimpleTransmission</type>
+            <joint name="${name}_twist_joint">
+            <hardwareInterface>hardware_interface/EffortJointInterface</hardwareInterface>
+            </joint>
+            <actuator name="${name}_twist_motor">
+            <hardwareInterface>hardware_interface/EffortJointInterface</hardwareInterface>
+            <mechanicalReduction>1</mechanicalReduction>
+            </actuator>
+        </transmission>
+        <transmission name="${name}_shoulder_tran">
+            <type>transmission_interface/SimpleTransmission</type>
+            <joint name="${name}_shoulder_joint">
+            <hardwareInterface>hardware_interface/EffortJointInterface</hardwareInterface>
+            </joint>
+            <actuator name="${name}_shoulder_motor">
+            <hardwareInterface>hardware_interface/EffortJointInterface</hardwareInterface>
+            <mechanicalReduction>1</mechanicalReduction>
+            </actuator>
+        </transmission>
+        <transmission name="${name}_elbow_tran">
+            <type>transmission_interface/SimpleTransmission</type>
+            <joint name="${name}_elbow_joint">
+            <hardwareInterface>hardware_interface/EffortJointInterface</hardwareInterface>
+            </joint>
+            <actuator name="${name}_twist_motor">
+            <hardwareInterface>hardware_interface/EffortJointInterface</hardwareInterface>
+            <mechanicalReduction>1</mechanicalReduction>
+            </actuator>
+        </transmission>
+    </xacro:macro>
 </robot>
