Commit message: humanoid model

File: Hector_ROS_Simulation/hector_description/xacro/const.xacro (robot description, xacro)
@@ -217,3 +217,90 @@
     <xacro:property name="toe_iyz" value="0.0"/>
     <xacro:property name="toe_izz" value="0.000249491"/>
+    <!-- twist -->
+    <!-- joint -->
+    <xacro:property name="twist_offset_x" value="0.0"/>
+    <xacro:property name="twist_offset_y" value="0.0"/>
+    <xacro:property name="twist_offset_z" value="-0.22"/>
+    <xacro:property name="twist_offset" value="0.019"/>
+    <xacro:property name="twist_max" value="1.4"/>
+    <xacro:property name="twist_min" value="-1.4"/>
+    <xacro:property name="twist_velocity_max" value="21"/>
+    <xacro:property name="twist_torque_max" value="33.5"/>
+    <!-- collision -->
+    <xacro:property name="twist_x" value="0.01"/>
+    <xacro:property name="twist_y" value="0.0194"/>
+    <xacro:property name="twist_z" value="-0.02"/>
+    <xacro:property name="twist_length" value="0.25"/>
+    <xacro:property name="twist_width" value="0.034"/>
+    <xacro:property name="twist_height" value="0.043"/>
+    <xacro:property name="twist_radius" value="0.041"/>
+    <xacro:property name="twist_length" value="0.08"/>
+    <!-- inertial -->
+    <!-- <xacro:property name="twist_mass" value="1.096"/> -->
+    <xacro:property name="twist_mass" value="0.1096"/>
+    <xacro:property name="twist_com_x" value="-0.001568"/>
+    <xacro:property name="twist_com_y" value="-0.008134"/>
+    <xacro:property name="twist_com_z" value="0.000864"/>
+    <xacro:property name="twist_ixx" value="0.000822113"/>
+    <xacro:property name="twist_ixy" value="-0.000004982"/>
+    <xacro:property name="twist_ixz" value="-0.00003672"/>
+    <xacro:property name="twist_iyy" value="0.000983196"/>
+    <xacro:property name="twist_iyz" value="0.000002811"/>
+    <xacro:property name="twist_izz" value="0.000864753"/>
+    <!-- shoulder -->
+    <!-- joint -->
+    <xacro:property name="shoulder_offset_x" value="0.0"/>
+    <xacro:property name="shoulder_offset_y" value="0.0"/>
+    <xacro:property name="shoulder_offset_z" value="-0.22"/>
+    <xacro:property name="shoulder_max" value="1.4"/>
+    <xacro:property name="shoulder_min" value="-1.4"/>
+    <xacro:property name="shoulder_velocity_max" value="21"/>
+    <xacro:property name="shoulder_torque_max" value="33.5"/>
+    <!-- collision -->
+    <xacro:property name="shoulder_x" value="0.01"/>
+    <xacro:property name="shoulder_y" value="0.0194"/>
+    <xacro:property name="shoulder_z" value="-0.02"/>
+    <xacro:property name="shoulder_length" value="0.25"/>
+    <xacro:property name="shoulder_width" value="0.034"/>
+    <xacro:property name="shoulder_height" value="0.043"/>
+    <!-- inertial -->
+    <!-- <xacro:property name="shoulder_mass" value="1.528"/> -->
+    <xacro:property name="shoulder_mass" value="0.1528"/>
+    <xacro:property name="shoulder_com_x" value="-0.000482"/>
+    <xacro:property name="shoulder_com_y" value="0.02001"/>
+    <xacro:property name="shoulder_com_z" value="-0.031996"/>
+    <xacro:property name="shoulder_ixx" value="0.00991611"/>
+    <xacro:property name="shoulder_ixy" value="0.000010388"/>
+    <xacro:property name="shoulder_ixz" value="0.000250428"/>
+    <xacro:property name="shoulder_iyy" value="0.009280083"/>
+    <xacro:property name="shoulder_iyz" value="-0.00008511"/>
+    <xacro:property name="shoulder_izz" value="0.00178256"/>
+    <!-- elbow -->
+    <!-- joint -->
+    <xacro:property name="elbow_offset_x" value="0.0"/>
+    <xacro:property name="elbow_offset_y" value="0.0"/>
+    <xacro:property name="elbow_offset_z" value="-0.22"/>
+    <xacro:property name="elbow_max" value="1.4"/>
+    <xacro:property name="elbow_min" value="-1.4"/>
+    <xacro:property name="elbow_velocity_max" value="21"/>
+    <xacro:property name="elbow_torque_max" value="33.5"/>
+    <!-- collision -->
+    <xacro:property name="elbow_x" value="0.01"/>
+    <xacro:property name="elbow_y" value="0.0194"/>
+    <xacro:property name="elbow_z" value="-0.02"/>
+    <xacro:property name="elbow_length" value="0.25"/>
+    <xacro:property name="elbow_width" value="0.016"/>
+    <xacro:property name="elbow_height" value="0.016"/>
+    <!-- inertial -->
+    <!-- <xacro:property name="elbow_mass" value="0.241"/> -->
+    <xacro:property name="elbow_mass" value="0.0241"/>
+    <xacro:property name="elbow_com_x" value="-0.002196"/>
+    <xacro:property name="elbow_com_y" value="-0.000381"/>
+    <xacro:property name="elbow_com_z" value="-0.12338"/>
+    <xacro:property name="elbow_ixx" value="0.006181961"/>
+    <xacro:property name="elbow_ixy" value="0.000000237"/>
+    <xacro:property name="elbow_ixz" value="-0.000002985"/>
+    <xacro:property name="elbow_iyy" value="0.006196546"/>
+    <xacro:property name="elbow_iyz" value="0.000005138"/>
+    <xacro:property name="elbow_izz" value="0.000034774"/>
 </robot>

File: Hector_ROS_Simulation/hector_description/xacro/robot.xacro (robot description, xacro)
@@ -4,4 +4,5 @@
     <xacro:include filename="$(find hector_description)/xacro/materials.xacro"/>
     <xacro:include filename="$(find hector_description)/xacro/leg.xacro"/>
+    <xacro:include filename="$(find hector_description)/xacro/arm.xacro"/>
     <xacro:include filename="$(find hector_description)/xacro/stairs.xacro"/>
     <xacro:include filename="$(find hector_description)/xacro/gazebo.xacro"/>
@@ -114,3 +115,9 @@
         <origin rpy="0 0 0" xyz="${hip_offset_x} ${-hip_offset_y} ${-hip_offset_z}"/>
     </xacro:leg>
+    <xacro:arm name="L" mirror="1" mirror_dae="False">
+        <origin rpy="0 0 0" xyz="${hip_offset_x} ${hip_offset_y} ${-hip_offset_z}"/>
+    </xacro:arm>
+    <xacro:arm name="R" mirror="-1" mirror_dae="True">
+        <origin rpy="0 0 0" xyz="${hip_offset_x} ${-hip_offset_y} ${-hip_offset_z}"/>
+    </xacro:arm>
 </robot>

Commit message: model physical parameter update

File: Hector_ROS_Simulation/hector_description/xacro/const.xacro (robot description, xacro)
@@ -18,11 +18,11 @@
     <xacro:property name="trunk_com_y" value="0.0"/>
     <xacro:property name="trunk_com_z" value="0.0"/>
-    <xacro:property name="trunk_mass" value="5.7"/>
-    <xacro:property name="trunk_ixx" value="0.0463619"/>
+    <xacro:property name="trunk_mass" value="4.87"/>
+    <xacro:property name="trunk_ixx" value="0.052"/>
     <xacro:property name="trunk_ixy" value="0.0"/>
     <xacro:property name="trunk_ixz" value="0.0"/>
-    <xacro:property name="trunk_iyy" value="0.036636"/>
+    <xacro:property name="trunk_iyy" value="0.0441"/>
     <xacro:property name="trunk_iyz" value="0.0"/>
-    <xacro:property name="trunk_izz" value="0.024569"/>
+    <xacro:property name="trunk_izz" value="0.0184"/>
     <!-- hip value -->
     <!-- joint -->
@@ -30,6 +30,6 @@
     <xacro:property name="hip_offset_y" value="0.047"/>
     <xacro:property name="hip_offset_z" value="0.1265"/>
-    <xacro:property name="hip_max" value="30"/>
-    <xacro:property name="hip_min" value="-30"/>
+    <xacro:property name="hip_max" value="45"/>
+    <xacro:property name="hip_min" value="-45"/>
     <xacro:property name="hip_velocity_max" value="21"/>
     <xacro:property name="hip_torque_max" value="33.5"/>
@@ -42,14 +42,14 @@
     <xacro:property name="hip_height" value="0.0001"/>
     <!-- inertial -->
-    <xacro:property name="hip_com_x" value="0.025109"/>
-    <xacro:property name="hip_com_y" value="-0.002292"/>
-    <xacro:property name="hip_com_z" value="-0.024732"/>
-    <xacro:property name="hip_mass" value="0.224"/>
-    <xacro:property name="hip_ixx" value="0.000002104"/>
+    <xacro:property name="hip_com_x" value="0.0268"/>
+    <xacro:property name="hip_com_y" value="-0.00315"/>
+    <xacro:property name="hip_com_z" value="-0.0272"/>
+    <xacro:property name="hip_mass" value="0.173"/>
+    <xacro:property name="hip_ixx" value="0.00022"/>
     <xacro:property name="hip_ixy" value="0.0"/>
     <xacro:property name="hip_ixz" value="0.0"/>
-    <xacro:property name="hip_iyy" value="0.000005354"/>
+    <xacro:property name="hip_iyy" value="0.00024"/>
     <xacro:property name="hip_iyz" value="0.0"/>
-    <xacro:property name="hip_izz" value="0.000007416"/>
+    <xacro:property name="hip_izz" value="0.00016"/>
     <!-- hip_trans value -->
     <!-- joint -->
@@ -61,11 +61,11 @@
     <xacro:property name="hip_trans_radius" value="0.045"/>
     <!-- inertial -->
-    <xacro:property name="hip_trans_mass" value="0.65"/>
-    <xacro:property name="hip_trans_ixx" value="0.00043875"/>
+    <xacro:property name="hip_trans_mass" value="0.605"/>
+    <xacro:property name="hip_trans_ixx" value="0.00048"/>
     <xacro:property name="hip_trans_ixy" value="0.0"/>
     <xacro:property name="hip_trans_ixz" value="0.0"/>
-    <xacro:property name="hip_trans_iyy" value="0.00043875"/>
+    <xacro:property name="hip_trans_iyy" value="0.00048"/>
     <xacro:property name="hip_trans_iyz" value="0.0"/>
-    <xacro:property name="hip_trans_izz" value="0.000658125"/>
+    <xacro:property name="hip_trans_izz" value="0.00071"/>
     <!-- hip2 value -->
     <!-- joint -->
@@ -73,6 +73,6 @@
     <xacro:property name="hip2_offset_y" value="0.015"/>
     <xacro:property name="hip2_offset_z" value="0.0705"/>
-    <xacro:property name="hip2_max" value="30"/>
-    <xacro:property name="hip2_min" value="-30"/>
+    <xacro:property name="hip2_max" value="45"/>
+    <xacro:property name="hip2_min" value="-45"/>
     <xacro:property name="hip2_velocity_max" value="21"/>
     <xacro:property name="hip2_torque_max" value="33.5"/>
@@ -82,11 +82,11 @@
     <xacro:property name="hip2_height" value="0.00001"/>
     <!-- inertial -->
-    <xacro:property name="hip2_mass" value="0.095"/>
-    <xacro:property name="hip2_ixx" value="0.000051083"/>
+    <xacro:property name="hip2_mass" value="0.0722"/>
+    <xacro:property name="hip2_ixx" value="0.00004"/>
     <xacro:property name="hip2_ixy" value="0.0"/>
     <xacro:property name="hip2_ixz" value="0.0"/>
-    <xacro:property name="hip2_iyy" value="0.0000139825"/>
+    <xacro:property name="hip2_iyy" value="0.000101"/>
     <xacro:property name="hip2_iyz" value="0.0"/>
-    <xacro:property name="hip2_izz" value="0.000093473"/>
+    <xacro:property name="hip2_izz" value="0.00007"/>
     <!-- hip2_trans value -->
     <!-- joint -->
@@ -98,11 +98,11 @@
     <xacro:property name="hip2_trans_radius" value="0.045"/>
     <!-- inertial -->
-    <xacro:property name="hip2_trans_mass" value="0.65"/>
-    <xacro:property name="hip2_trans_ixx" value="0.00043875"/>
+    <xacro:property name="hip2_trans_mass" value="0.605"/>
+    <xacro:property name="hip2_trans_ixx" value="0.00048"/>
     <xacro:property name="hip2_trans_ixy" value="0.0"/>
     <xacro:property name="hip2_trans_ixz" value="0.0"/>
-    <xacro:property name="hip2_trans_iyy" value="0.00043875"/>
+    <xacro:property name="hip2_trans_iyy" value="0.00048"/>
     <xacro:property name="hip2_trans_iyz" value="0.0"/>
-    <xacro:property name="hip2_trans_izz" value="0.000658125"/>
+    <xacro:property name="hip2_trans_izz" value="0.00071"/>
     <!-- thigh -->
     <!-- joint -->
@@ -110,6 +110,6 @@
     <xacro:property name="thigh_offset_y" value="0.018"/>
     <xacro:property name="thigh_offset_z" value="0"/>
-    <xacro:property name="thigh_max" value="3.14"/>
-    <xacro:property name="thigh_min" value="-3.14"/>
+    <xacro:property name="thigh_max" value="100"/>
+    <xacro:property name="thigh_min" value="-100"/>
     <xacro:property name="thigh_velocity_max" value="21"/>
     <xacro:property name="thigh_torque_max" value="33.5"/>
@@ -122,14 +122,14 @@
     <xacro:property name="thigh_height" value="0.18"/>
     <!-- inertial -->
-    <xacro:property name="thigh_mass" value="0.642"/>
+    <xacro:property name="thigh_mass" value="0.397"/>
     <xacro:property name="thigh_com_x" value="-0.000147"/>
     <xacro:property name="thigh_com_y" value="0.01991"/>
     <xacro:property name="thigh_com_z" value="-0.081117"/>
-    <xacro:property name="thigh_ixx" value="0.004437615"/>
+    <xacro:property name="thigh_ixx" value="0.0019"/>
     <xacro:property name="thigh_ixy" value="0.0"/>
     <xacro:property name="thigh_ixz" value="0.0"/>
-    <xacro:property name="thigh_iyy" value="0.004788512"/>
+    <xacro:property name="thigh_iyy" value="0.00218"/>
     <xacro:property name="thigh_iyz" value="0.0"/>
-    <xacro:property name="thigh_izz" value="0.000661818"/>
+    <xacro:property name="thigh_izz" value="0.00033"/>
     <!-- thigh1_trans value -->
     <!-- joint -->
@@ -141,11 +141,11 @@
     <xacro:property name="thigh1_trans_radius" value="0.045"/>
     <!-- inertial -->
-    <xacro:property name="thigh1_trans_mass" value="0.65"/>
-    <xacro:property name="thigh1_trans_ixx" value="0.00043875"/>
+    <xacro:property name="thigh1_trans_mass" value="0.605"/>
+    <xacro:property name="thigh1_trans_ixx" value="0.00048"/>
     <xacro:property name="thigh1_trans_ixy" value="0.0"/>
     <xacro:property name="thigh1_trans_ixz" value="0.0"/>
-    <xacro:property name="thigh1_trans_iyy" value="0.00043875"/>
+    <xacro:property name="thigh1_trans_iyy" value="0.00048"/>
     <xacro:property name="thigh1_trans_iyz" value="0.0"/>
-    <xacro:property name="thigh1_trans_izz" value="0.000658125"/>
+    <xacro:property name="thigh1_trans_izz" value="0.00071"/>
     <!-- thigh2_trans value -->
     <!-- joint -->
@@ -157,11 +157,11 @@
     <xacro:property name="thigh2_trans_radius" value="0.045"/>
     <!-- inertial -->
-    <xacro:property name="thigh2_trans_mass" value="0.65"/>
-    <xacro:property name="thigh2_trans_ixx" value="0.00043875"/>
+    <xacro:property name="thigh2_trans_mass" value="0.605"/>
+    <xacro:property name="thigh2_trans_ixx" value="0.00048"/>
     <xacro:property name="thigh2_trans_ixy" value="0.0"/>
     <xacro:property name="thigh2_trans_ixz" value="0.0"/>
-    <xacro:property name="thigh2_trans_iyy" value="0.00043875"/>
+    <xacro:property name="thigh2_trans_iyy" value="0.00048"/>
     <xacro:property name="thigh2_trans_iyz" value="0.0"/>
-    <xacro:property name="thigh2_trans_izz" value="0.000658125"/>
+    <xacro:property name="thigh2_trans_izz" value="0.00071"/>
     <!-- calf -->
     <!-- joint -->
@@ -169,8 +169,8 @@
     <xacro:property name="calf_offset_y" value="0.0"/>
     <xacro:property name="calf_offset_z" value="0.22"/>
-    <xacro:property name="calf_max" value="3.14"/>
-    <xacro:property name="calf_min" value="-3.14"/>
-    <xacro:property name="calf_velocity_max" value="21"/>
-    <xacro:property name="calf_torque_max" value="33.5"/>
+    <xacro:property name="calf_max" value="100"/>
+    <xacro:property name="calf_min" value="-100"/>
+    <xacro:property name="calf_velocity_max" value="14"/>
+    <xacro:property name="calf_torque_max" value="67"/>
     <!-- collision -->
     <xacro:property name="calf_x" value="0.0"/>
@@ -180,12 +180,12 @@
     <xacro:property name="calf_radius" value="0.015"/>
     <!-- inertial -->
-    <xacro:property name="calf_mass" value="0.303"/>
+    <xacro:property name="calf_mass" value="0.163"/>
     <xacro:property name="calf_com_x" value="0.0"/>
     <xacro:property name="calf_com_y" value="0.020417"/>
     <xacro:property name="calf_com_z" value="-0.1141"/>
-    <xacro:property name="calf_ixx" value="0.001911"/>
+    <xacro:property name="calf_ixx" value="0.00071"/>
     <xacro:property name="calf_ixy" value="0.0000"/>
     <xacro:property name="calf_ixz" value="0.0000"/>
-    <xacro:property name="calf_iyy" value="0.001910380"/>
+    <xacro:property name="calf_iyy" value="0.00071"/>
     <xacro:property name="calf_iyz" value="0.0"/>
     <xacro:property name="calf_izz" value="0.000068352"/>
@@ -195,6 +195,6 @@
     <xacro:property name="toe_offset_y" value="0.0"/>
     <xacro:property name="toe_offset_z" value="-0.22"/>
-    <xacro:property name="toe_max" value="1.4"/>
-    <xacro:property name="toe_min" value="-1.4"/>
+    <xacro:property name="toe_max" value="100"/>
+    <xacro:property name="toe_min" value="-100"/>
     <xacro:property name="toe_velocity_max" value="21"/>
     <xacro:property name="toe_torque_max" value="33.5"/>
@@ -207,13 +207,13 @@
     <xacro:property name="toe_height" value="0.04"/>
     <!-- inertial -->
-    <xacro:property name="toe_mass" value="0.214"/>
+    <xacro:property name="toe_mass" value="0.184"/>
     <xacro:property name="toe_com_x" value="0.010569"/>
     <xacro:property name="toe_com_y" value="0.017949"/>
     <xacro:property name="toe_com_z" value="-0.017118"/>
-    <xacro:property name="toe_ixx" value="0.000057298"/>
+    <xacro:property name="toe_ixx" value="0.00005"/>
     <xacro:property name="toe_ixy" value="0.0"/>
     <xacro:property name="toe_ixz" value="0.0"/>
-    <xacro:property name="toe_iyy" value="0.000290752"/>
+    <xacro:property name="toe_iyy" value="0.00021"/>
     <xacro:property name="toe_iyz" value="0.0"/>
-    <xacro:property name="toe_izz" value="0.000249491"/>
+    <xacro:property name="toe_izz" value="0.0002"/>
 </robot>

File: Hector_ROS_Simulation/hector_description/xacro/leg.xacro (robot description, xacro)
@@ -145,5 +145,5 @@
             <joint_properties damping="${damping}" friction="${friction}"/>
             <!-- <limit effort="${thigh_torque_max}" velocity="${thigh_velocity_max}"/> -->
-            <limit effort="${thigh_torque_max}" velocity="${thigh_velocity_max}" lower="${thigh_min}" upper="${thigh_max}"/>
+            <limit effort="${thigh_torque_max}" velocity="${thigh_velocity_max}" lower="${thigh_min*PI/180.0}" upper="${thigh_max*PI/180.0}"/>
         </joint>
         <link name="${name}_thigh">
@@ -227,5 +227,5 @@
             <axis xyz="0 1 0"/>
             <joint_properties damping="${damping}" friction="${friction}"/>
-            <limit effort="${calf_torque_max}" velocity="${calf_velocity_max}" lower="${calf_min}" upper="${calf_max}"/>
+            <limit effort="${calf_torque_max}" velocity="${calf_velocity_max}" lower="${calf_min*PI/180.0}" upper="${calf_max*PI/180.0}"/>
         </joint>
         <link name="${name}_calf">
@@ -265,5 +265,5 @@
             <axis xyz="0 1 0"/>
             <joint_properties damping="${damping}" friction="${friction}"/>
-            <limit effort="${toe_torque_max}" velocity="${toe_velocity_max}" lower="${toe_min}" upper="${toe_max}"/>
+            <limit effort="${toe_torque_max}" velocity="${toe_velocity_max}" lower="${toe_min*PI/180.0}" upper="${toe_max*PI/180.0}"/>
         </joint>
         <link name="${name}_toe">
